File: robko_PCB_arduino_shield/robko_PCB_arduino_shield/robko_PCB_arduino_shield.kicad_pcb (KiCad board)
At the start: 2 copper layers, 195.1 x 118.1 mm, 46 parts, among them J1 Barrel_Jack_Switch, J2 Conn_01x13_Male, J3 Conn_01x13_Male, J4 Conn_01x13_Male, U1 POLOLU_STEPPER_DRIVER, U2 POLOLU_STEPPER_DRIVER, U3 POLOLU_STEPPER_DRIVER, U4 POLOLU_STEPPER_DRIVER, U5 POLOLU_STEPPER_DRIVER, U6 POLOLU_STEPPER_DRIVER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

Commit message: подключены датчики; нужно вывести функцию нулевое положения; перейти от блокурующего runSpeedToPosition() к run()
Connections:
- J3 pad 3: M1_LIMIT -> M3_LIMIT
- J3 pad 4: M2_LIMIT -> M5_LIMIT
- J3 pad 5: M3_LIMIT -> M1_LIMIT
- J3 pad 7: M5_LIMIT -> M2_LIMIT
- R1 pad 1: M3_LIMIT -> M1_LIMIT
- R2 pad 1: M1_LIMIT -> M3_LIMIT
- R3 pad 1: M2_LIMIT -> M5_LIMIT
- R5 pad 1: M5_LIMIT -> M2_LIMIT
- SHIELD1 pad 42: M5_LIMIT -> M2_LIMIT
- SHIELD1 pad 44: M3_LIMIT -> M1_LIMIT
- SHIELD1 pad 45: M2_LIMIT -> M5_LIMIT
- SHIELD1 pad 46: M1_LIMIT -> M3_LIMIT
Routing:
- net M5_LIMIT: track 72.1 -> 66.2 mm
- net M2_LIMIT: track 66.2 -> 72.1 mm
