File: robko_PCB_arduino_shield/robko_PCB_arduino_shield/robko_PCB_arduino_shield.sch (KiCad schematic (older format))
At the start: 42 parts, among them J1 Barrel_Jack_Switch, J2 Conn_01x13_Male, J3 Conn_01x13_Male, J4 Conn_01x13_Male, U1 POLOLU_STEPPER_DRIVER, U2 POLOLU_STEPPER_DRIVER, U3 POLOLU_STEPPER_DRIVER, U4 POLOLU_STEPPER_DRIVER, U5 POLOLU_STEPPER_DRIVER, U6 POLOLU_STEPPER_DRIVER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

Commit message: подключены датчики; нужно вывести функцию нулевое положения; перейти от блокурующего runSpeedToPosition() к run()
Changed lines of the file:
@@
 $EndComp
 Text GLabel 14300 4450 2    50   Input ~ 0
-M1_LIMIT
+M3_LIMIT
 Wire Wire Line
 	14150 4450 14300 4450
 Text GLabel 14300 4550 2    50   Input ~ 0
-M2_LIMIT
+M5_LIMIT
 Wire Wire Line
 	14150 4550 14300 4550
 Text GLabel 14300 4650 2    50   Input ~ 0
-M3_LIMIT
+M1_LIMIT
 Wire Wire Line
 	14150 4650 14300 4650
@@
 	14150 4750 14300 4750
 Text GLabel 14300 4850 2    50   Input ~ 0
-M5_LIMIT
+M2_LIMIT
 Wire Wire Line
 	14150 4850 14300 4850
@@
 	14150 4950 14300 4950
 Text GLabel 350  6050 0    50   Input ~ 0
-M1_LIMIT
+M3_LIMIT
 Text GLabel 350  6150 0    50   Input ~ 0
-M2_LIMIT
+M5_LIMIT
 Text GLabel 350  6350 0    50   Input ~ 0
 M4_LIMIT
 Text GLabel 350  6450 0    50   Input ~ 0
-M5_LIMIT
+M2_LIMIT
 Text GLabel 350  6600 0    50   Input ~ 0
 M6_LIMIT
@@
 $EndComp
 Text GLabel 350  6250 0    50   Input ~ 0
-M3_LIMIT
+M1_LIMIT
 Wire Wire Line
 	350  6450 1550 6450

Commit message: PCB_Arduino_shield названы a4998
Parts:
- SHIELD1: symbol arduino_shieldsNCL:ARDUINO_MEGA_SHIELD -> robko_PCB_arduino_shield-rescue:ARDUINO_MEGA_SHIELD-arduino_shieldsNCL
- a4988_1: renamed from U1; symbol sb-cnc-shield-rescue:POLOLU_STEPPER_DRIVER -> robko_PCB_arduino_shield-rescue:POLOLU_STEPPER_DRIVER-sb-cnc-shield-rescue
- a4988_2: renamed from U2; symbol sb-cnc-shield-rescue:POLOLU_STEPPER_DRIVER -> robko_PCB_arduino_shield-rescue:POLOLU_STEPPER_DRIVER-sb-cnc-shield-rescue
- a4988_3: renamed from U3; symbol sb-cnc-shield-rescue:POLOLU_STEPPER_DRIVER -> robko_PCB_arduino_shield-rescue:POLOLU_STEPPER_DRIVER-sb-cnc-shield-rescue
- a4988_4: renamed from U4; symbol sb-cnc-shield-rescue:POLOLU_STEPPER_DRIVER -> robko_PCB_arduino_shield-rescue:POLOLU_STEPPER_DRIVER-sb-cnc-shield-rescue
- a4988_5: renamed from U5; symbol sb-cnc-shield-rescue:POLOLU_STEPPER_DRIVER -> robko_PCB_arduino_shield-rescue:POLOLU_STEPPER_DRIVER-sb-cnc-shield-rescue
- a4988_6: renamed from U6; symbol sb-cnc-shield-rescue:POLOLU_STEPPER_DRIVER -> robko_PCB_arduino_shield-rescue:POLOLU_STEPPER_DRIVER-sb-cnc-shield-rescue
Other:
- moved on the sheet: C1, C2, C3, C4, C5, C6, J1, J2, J3, J4, R1, R2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
